Commit message: Ewha-glab up-to-date

File: robotiq_3f_gripper_visualization/cfg/robotiq-3f-gripper_articulated.urdf (robot description, URDF)
Before this commit: robot robotiq-3f-gripper_articulated, 13 links, 12 joints
Links:
- link finger_1_link_3: geometry visual mesh filename=package://robotiq_3f_gripper_visualization/meshes/robotiq-3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
- link finger_2_link_3: geometry visual mesh filename=package://robotiq_3f_gripper_visualization/meshes/robotiq-3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
- link finger_middle_link_3: geometry visual mesh filename=package://robotiq_3f_gripper_visualization/meshes/robotiq-3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

File: robotiq_3f_gripper_visualization/cfg/robotiq-3f-gripper_articulated_macro.xacro (robot description, xacro)
@@ -35,4 +35,5 @@
     		</gazebo>
 		<link name="${prefix}gripper_tool0"/>
+		<link name="${prefix}pen_tool0"/>
         <inertial>
             <origin xyz="0 0 0" rpy="0 0 0"/>
@@ -53,5 +54,5 @@
 			<child link="${prefix}finger_2_link_0"/>
 			<axis xyz="0 1 0"/>
-			<origin xyz="-0.0455 0.0214 -0.036" rpy="0 3.1416 -1.57"/>
+			<origin xyz="-0.0455 0.0214 -0.036" rpy="0 ${pi} -1.57"/>
 			<limit lower="-0.192" upper="0.1784" effort="100" velocity="100"/>
 		</joint>
@@ -65,5 +66,11 @@
 			<parent link="${prefix}palm"/>
 			<child link="${prefix}gripper_tool0"/>
-			<origin xyz="0.0 0.0875 0.0" rpy="0 0 1.5707"/>
+			<!--origin xyz="0.0 0.0875 0.0" rpy="0 0 1.5707"/-->
+			<origin xyz="0.0 0.18 0.0" rpy="0 0 1.5707"/>
+		</joint>
+		<joint name="${prefix}pen" type="fixed">
+			<parent link="${prefix}gripper_tool0"/>
+			<child link="${prefix}pen_tool0"/>
+			<origin xyz="-0.065 0.0 -0.17" rpy="0 0 ${(-PI/2)}"/>
 		</joint>
 		<!-- end of joint list -->

File: robotiq_3f_gripper_visualization/cfg/robotiq-3f-gripper_finger_articulated_macro.xacro (robot description, xacro)
@@ -93,5 +93,5 @@
 	      		<mu2>1.1</mu2>
 	    	</gazebo>
-		<link name="${prefix}link_3">
+		<link name="${prefix}link_3">link name="${prefix}link_3">
 			<visual>
 				<origin xyz="0 0 0" rpy="0 0 0.52"/>
@@ -101,4 +101,5 @@
 				<material name="gray"/>
 			</visual>
+			<!--
 			<collision>
 				<origin xyz="0 0 0" rpy="0 0 0.52"/>
@@ -108,4 +109,5 @@
 				<material name="yellow"/>
 			</collision>
+			-->
             <inertial>
                 <origin xyz="0 0 0" rpy="0 0 0"/>

Commit message: Add files for dual arm

File: robotiq_3f_gripper_visualization/cfg/robotiq-3f-gripper_articulated.urdf (robot description, URDF)
Before this commit: robot robotiq-3f-gripper_articulated, 13 links, 12 joints
Links:
- link finger_1_link_3: geometry visual mesh filename=package://robotiq_3f_gripper_visualization/meshes/robotiq-3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
- link finger_2_link_3: geometry visual mesh filename=package://robotiq_3f_gripper_visualization/meshes/robotiq-3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
- link finger_middle_link_3: geometry visual mesh filename=package://robotiq_3f_gripper_visualization/meshes/robotiq-3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

File: robotiq_3f_gripper_visualization/cfg/robotiq-3f-gripper_articulated_macro.xacro (robot description, xacro)
@@ -30,5 +30,10 @@
 			</collision>
 		</link>
-		<link name="${prefix}tool0"/>
+		<gazebo reference="${prefix}palm">
+      		<mu1>1.1</mu1>
+      		<mu2>1.1</mu2>
+    		</gazebo>
+		<link name="${prefix}gripper_tool0"/>
+		<link name="${prefix}pen_tool0"/>
         <inertial>
             <origin xyz="0 0 0" rpy="0 0 0"/>
@@ -49,5 +54,5 @@
 			<child link="${prefix}finger_2_link_0"/>
 			<axis xyz="0 1 0"/>
-			<origin xyz="-0.0455 0.0214 -0.036" rpy="0 3.1416 -1.57"/>
+			<origin xyz="-0.0455 0.0214 -0.036" rpy="0 ${pi} -1.57"/>
 			<limit lower="-0.192" upper="0.1784" effort="100" velocity="100"/>
 		</joint>
@@ -60,8 +65,32 @@
 		<joint name="${prefix}palm_tool0" type="fixed">
 			<parent link="${prefix}palm"/>
-			<child link="${prefix}tool0"/>
-			<origin xyz="0.0 0.0875 0.0" rpy="0 0 1.5707"/>
+			<child link="${prefix}gripper_tool0"/>
+			<!--origin xyz="0.0 0.0875 0.0" rpy="0 0 1.5707"/-->
+			<origin xyz="0.0 0.18 0.0" rpy="0 0 1.5707"/>
+		</joint>
+		<joint name="${prefix}pen" type="fixed">
+			<parent link="${prefix}gripper_tool0"/>
+			<child link="${prefix}pen_tool0"/>
+			<origin xyz="-0.065 0.0 -0.17" rpy="0 0 ${(-PI/2)}"/>
 		</joint>
 		<!-- end of joint list -->
+		<transmission name="${prefix}palm_finger_1_trans">
+      			<type>transmission_interface/SimpleTransmission</type>
+		        <joint name="${prefix}palm_finger_1_joint">
+			 <hardwareInterface>hardware_interface/PositionJointInterface</hardwareInterface>
+		        </joint>
+		        <actuator name="${prefix}palm_finger_1_motor">
+			 <mechanicalReduction>1</mechanicalReduction>
+		        </actuator>
+	 	</transmission>
+	        <transmission name="${prefix}palm_finger_2_trans">
+	          <type>transmission_interface/SimpleTransmission</type>
+	          <joint name="${prefix}palm_finger_2_joint">
+	    	<hardwareInterface>hardware_interface/PositionJointInterface</hardwareInterface>
+	          </joint>
+	          <actuator name="${prefix}palm_finger_2_motor">
+	      	    <mechanicalReduction>1</mechanicalReduction>
+	          </actuator>
+	       </transmission>
 	</xacro:macro>
 </robot>

File: robotiq_3f_gripper_visualization/cfg/robotiq-3f-gripper_finger_articulated_macro.xacro (robot description, xacro)
@@ -7,4 +7,5 @@
 <robot xmlns:xacro="http://ros.org/wiki/xacro">
         <xacro:macro name="robotiq-3f-gripper_finger_articulated" params="prefix">
+		<xacro:include filename="$(find robotiq_3f_gripper_visualization)/cfg/robotiq.transmission.xacro" />
 		<!-- link list -->
 		<link name="${prefix}link_0">
@@ -33,4 +34,8 @@
             </inertial>
 		</link>
+		<gazebo reference="${prefix}link_0">
+	      		<mu1>1.1</mu1>
+	      		<mu2>1.1</mu2>
+	    	</gazebo>
 		<link name="${prefix}link_1">
 			<visual>
@@ -54,4 +59,8 @@
             </inertial>
 		</link>
+		<gazebo reference="${prefix}link_1">
+	      		<mu1>1.1</mu1>
+	      		<mu2>1.1</mu2>
+	    	</gazebo>
 		<link name="${prefix}link_2">
 			<!--
@@ -80,5 +89,9 @@
             </inertial>
 		</link>
-		<link name="${prefix}link_3">
+		<gazebo reference="${prefix}link_2">
+	      		<mu1>1.1</mu1>
+	      		<mu2>1.1</mu2>
+	    	</gazebo>
+		<link name="${prefix}link_3">link name="${prefix}link_3">
 			<visual>
 				<origin xyz="0 0 0" rpy="0 0 0.52"/>
@@ -88,4 +101,5 @@
 				<material name="gray"/>
 			</visual>
+			<!--
 			<collision>
 				<origin xyz="0 0 0" rpy="0 0 0.52"/>
@@ -95,4 +109,5 @@
 				<material name="yellow"/>
 			</collision>
+			-->
             <inertial>
                 <origin xyz="0 0 0" rpy="0 0 0"/>
@@ -101,6 +116,11 @@
             </inertial>
 		</link>
+		<gazebo reference="${prefix}link_3">
+	      		<mu1>1.1</mu1>
+	      		<mu2>1.1</mu2>
+	    	</gazebo>
 		<!-- end of link list -->
 		<!-- joint list -->
+		<xacro:robotiq_transmission prefix="${prefix}" />
 		<joint name="${prefix}joint_1" type="revolute">
 			<parent link="${prefix}link_0"/>
